File: img/clk.sch (EAGLE design)
At the start: 27 parts, among them IC1 MEGA8-P, IC2 DS1307, J1 22-27-2021-02

Commit message: Finished and tested version 2
Parts:
- removed J1: 22-27-2021-02, con-molex:22-27-2021-02
- removed JP1: (no value), adafruit:PINHD-1X1
- added C3: (no value), rcl:C-EU025-024X044
- added JP2: (no value), pinhead:PINHD-1X3
- added S1, S2, S3: DTS-6, switch-tact:DTS-6
- R10, R11, R12, R13, R14, R7, R8, R9: device rcl:R-EU_0207/2V -> rcl:R-EU_0204/2V
Connections:
- removed net N$13: IC1.PC6(/RESET), R15.1
- new net BUTTON_1: IC1.PD0(RXD), S1.3, S1.4
- new net BUTTON_2: IC1.PD1(TXD), S2.3, S2.4
- new net BUTTON_3: IC1.PD2(INT0), S3.3, S3.4
- new net N$24: IC1.PB4(MISO), R14.1
- new net N$25: IC1.PC3(ADC3), R15.2
- net +5V: now also JP2.2; no longer J1-1.S, R15.2
- net A: now also R9.2; no longer R11.1
- net B: now also R7.2; no longer R12.1
- net C: now also R13.2; no longer R14.1
- net D: now also R11.2; no longer R13.1
- net DP: now also R12.2; no longer R8.1
- net E: now also R10.2; no longer R9.1
- net F: now also R8.2; no longer R10.1
- net G: now also R14.2; no longer R7.1
- net GND: now also C3.1, IC2.VBAT, JP2.3, S1.1, S1.2, S2.1, S2.2, S3.1, S3.2; no longer J1-2.S
- net N$14: now also IC1.PC1(ADC1); no longer IC1.PB2(SS/OC1B)
- net N$15: now also IC1.PD3(INT1); no longer IC1.PB3(MOSI/OC2)
- net N$16: now also IC1.PD5(T1), R7.1; no longer IC1.PB4(MISO), R6.1
- net N$17: now also IC1.PD6(AIN0), R8.1; no longer IC1.PC3(ADC3), R10.2
- net N$18: now also IC1.PD7(AIN1), R9.1; no longer IC1.PD1(TXD), R11.2
- net N$19: now also IC1.PB0(ICP), R10.1; no longer IC1.PD2(INT0), R12.2
- net N$20: now also IC1.PB1(OC1A), R11.1; no longer IC1.PD3(INT1), R13.2
- net N$21: now also IC1.PB2(SS/OC1B), R12.1; no longer IC1.PD4(XCK/T0), R14.2
- net N$22: now also IC1.PB3(MOSI/OC2), R13.1; no longer IC1.PB1(OC1A), R3.1
- net N$3: now also C3.2, IC1.AREF; no longer IC1.PC0(ADC0), R7.2
- net N$4: now also JP2.1, R15.1; no longer IC1.PC1(ADC1), R8.2
- net N$7: now also IC1.PC0(ADC0), R6.1; no longer IC2.VBAT, JP1.1
- net N$8: now also IC1.PD4(XCK/T0), R3.1; no longer IC1.PC2(ADC2), R9.2
Other:
- moved on the sheet: IC2, Q1, R1, R10, R11, R12, R13, R14, R15, R2, R7, R8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
